Commit message: Generating correct inertia values for object now

File: cw3_description/urdf/weighted_object.xacro (robot description, xacro)
@@ -3,11 +3,14 @@
   <xacro:include filename="$(find iiwa_fri_description)/urdf/utilities.xacro" />
   <xacro:macro name="weighted_object" params="mass">
+   <xacro:property name="height" value="0.1" />
+   <xacro:property name="length" value="0.1" />
+   <xacro:property name="width" value="0.1" />
     <link name="object_link_0">
       <inertial>
         <origin xyz="0.0 0.0 0.05" rpy="0 0 0"/>
         <mass value="${mass}"/>
-        <inertia ixx="0.1"
-             iyy="0.1"
-             izz="0.1"
+        <inertia ixx="${mass * (height * height + length * length) / 12}"
+             iyy="${mass * (width * width + length * length) / 12}"
+             izz="${mass * (width * width + height * height) / 12}"
              ixy="0" iyz="0" ixz="0"/>
       </inertial>
