Commit message: controller tuned and working, occasionally a bit shaky during the motion but gets to the desired position

File: iiwa_fri_description/urdf/iiwa14.xacro (robot description, xacro)
@@ -12,5 +12,5 @@
   <xacro:property name="safety_controller_k_vel" value="2" />
   <xacro:property name="joint_damping" value="0.5" />
-  <xacro:property name="max_effort" value="300"/>
+  <xacro:property name="max_effort" value="3000"/>
   <xacro:property name="max_velocity" value="10"/>
   <xacro:macro name="iiwa14" params="hardware_interface robot_name">
@@ -50,8 +50,4 @@
       <limit lower="${-170 * PI / 180}" upper="${170 * PI / 180}"
              effort="${max_effort}" velocity="${max_velocity}" />
-      <safety_controller soft_lower_limit="${-168 * PI / 180}"
-                         soft_upper_limit="${168 * PI / 180}"
-                         k_position="${safety_controller_k_pos}"
-                         k_velocity="${safety_controller_k_vel}"/>
       <dynamics damping="${joint_damping}"/>
     </joint>
@@ -85,8 +81,4 @@
       <limit lower="${-120 * PI / 180}" upper="${120 * PI / 180}"
              effort="${max_effort}" velocity="${max_velocity}" />
-      <safety_controller soft_lower_limit="${-118 * PI / 180}"
-                         soft_upper_limit="${118 * PI / 180}"
-                         k_position="${safety_controller_k_pos}"
-                         k_velocity="${safety_controller_k_vel}"/>
       <dynamics damping="${joint_damping}"/>
     </joint>
@@ -120,8 +112,4 @@
       <limit lower="${-170 * PI / 180}" upper="${170 * PI / 180}"
              effort="${max_effort}" velocity="${max_velocity}" />
-      <safety_controller soft_lower_limit="${-168 * PI / 180}"
-                         soft_upper_limit="${168 * PI / 180}"
-                         k_position="${safety_controller_k_pos}"
-                         k_velocity="${safety_controller_k_vel}"/>
       <dynamics damping="${joint_damping}"/>
     </joint>
@@ -155,8 +143,4 @@
       <limit lower="${-120 * PI / 180}" upper="${120 * PI / 180}"
              effort="${max_effort}" velocity="${max_velocity}" />
-      <safety_controller soft_lower_limit="${-118 * PI / 180}"
-                         soft_upper_limit="${118 * PI / 180}"
-                         k_position="${safety_controller_k_pos}"
-                         k_velocity="${safety_controller_k_vel}"/>
       <dynamics damping="${joint_damping}"/>
     </joint>
@@ -190,8 +174,4 @@
       <limit lower="${-170 * PI / 180}" upper="${170 * PI / 180}"
              effort="${max_effort}" velocity="${max_velocity}" />
-      <safety_controller soft_lower_limit="${-168 * PI / 180}"
-                         soft_upper_limit="${168 * PI / 180}"
-                         k_position="${safety_controller_k_pos}"
-                         k_velocity="${safety_controller_k_vel}"/>
       <dynamics damping="${joint_damping}"/>
     </joint>
@@ -225,8 +205,4 @@
       <limit lower="${-120 * PI / 180}" upper="${120 * PI / 180}"
              effort="${max_effort}" velocity="${max_velocity}" />
-      <safety_controller soft_lower_limit="${-118 * PI / 180}"
-                         soft_upper_limit="${118 * PI / 180}"
-                         k_position="${safety_controller_k_pos}"
-                         k_velocity="${safety_controller_k_vel}"/>
       <dynamics damping="${joint_damping}"/>
     </joint>
@@ -260,8 +236,4 @@
       <limit lower="${-175 * PI / 180}" upper="${175 * PI / 180}"
              effort="${max_effort}" velocity="${max_velocity}" />
-      <safety_controller soft_lower_limit="${-173 * PI / 180}"
-                         soft_upper_limit="${173 * PI / 180}"
-                         k_position="${safety_controller_k_pos}"
-                         k_velocity="${safety_controller_k_vel}"/>
       <dynamics damping="${joint_damping}"/>
     </joint>
